File: OSHW_STEPPER_DRIVER.brd (EAGLE design)
At the start: 104.3 x 79.2 mm, 63 parts, among them X2 MSTBA2, X3 MSTBA4

Commit message: rework of some GND signals, added version text on PCB
Other:
- board size 104.3 x 79.2 mm -> 104.4 x 79.2 mm
- board text added: "v0.6.1"
Changed lines of the file:
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@@
 <setting verticaltext="up"/>
 </settings>
-<grid distance="0.01" unitdist="inch" unit="mm" style="lines" multiple="1" display="yes" altdistance="0.01" altunitdist="inch" altunit="mm"/>
+<grid distance="0.01" unitdist="mm" unit="mm" style="lines" multiple="1" display="yes" altdistance="0.01" altunitdist="mm" altunit="mm"/>
 <layers>
 <layer number="1" name="Top" color="4" fill="1" visible="yes" active="yes"/>
@@
 <plain>
 <wire x1="0" y1="0" x2="104.318" y2="0" width="0" layer="20"/>
-<wire x1="104.318" y1="0" x2="104.318" y2="79.176" width="0" layer="20"/>
-<wire x1="104.318" y1="79.176" x2="0.1" y2="79.086" width="0" layer="20"/>
-<wire x1="0.1" y1="79.086" x2="0" y2="0" width="0" layer="20"/>
+<wire x1="104.318" y1="0" x2="104.348" y2="79.156" width="0" layer="20"/>
+<wire x1="104.348" y1="79.156" x2="-0.02" y2="79.186" width="0" layer="20"/>
+<wire x1="-0.02" y1="79.186" x2="0" y2="0" width="0" layer="20"/>
 <text x="86.36" y="21.082" size="2.54" layer="25" rot="R90">oshw.it</text>
+<text x="10.73" y="73.87" size="1.778" layer="21">v0.6.1</text>
 </plain>
 <attributes>
@@
 <vertex x="0.254" y="78.74"/>
 <vertex x="0.254" y="62.738"/>
-<vertex x="17.526" y="62.23"/>
-<vertex x="17.78" y="49.784"/>
-<vertex x="80.772" y="49.784"/>
-<vertex x="80.78" y="13.506"/>
-<vertex x="96.258" y="10.72"/>
-<vertex x="96.198" y="0.412"/>
+<vertex x="-0.254" y="-2.286"/>
+<vertex x="28.448" y="-5.334"/>
+<vertex x="81.534" y="-3.556"/>
+<vertex x="99.322" y="-3.512"/>
+<vertex x="107.688" y="-2.996"/>
+<vertex x="110.676" y="-2.636"/>
 <vertex x="104.394" y="0.254"/>
 <vertex x="104.648" y="4.064"/>
@@
 <wire x1="21.59" y1="73.914" x2="21.59" y2="71.374" width="0.254" layer="1"/>
 <wire x1="21.59" y1="71.374" x2="21.59" y2="68.834" width="0.254" layer="1"/>
-<wire x1="21.59" y1="68.834" x2="9.398" y2="68.834" width="0.4064" layer="1"/>
-<wire x1="9.398" y1="68.834" x2="6.096" y2="65.532" width="0.4064" layer="1"/>
+<wire x1="21.59" y1="68.834" x2="18.818" y2="65.514" width="0.4064" layer="1"/>
+<wire x1="18.818" y1="65.514" x2="6.096" y2="65.532" width="0.4064" layer="1"/>
 <wire x1="69.292" y1="70.402" x2="71.44" y2="72.55" width="0.254" layer="1"/>
 <wire x1="71.44" y1="72.55" x2="76.454" y2="72.55" width="0.254" layer="1"/>
@@
 <wire x1="54.3" y1="66.55" x2="53.34" y2="67.51" width="0.4064" layer="1"/>
 <wire x1="53.34" y1="67.51" x2="53.34" y2="70.358" width="0.4064" layer="1"/>
-<polygon width="0.254" layer="16">
-<vertex x="0" y="61.976"/>
-<vertex x="17.018" y="61.976"/>
-<vertex x="17.272" y="61.722"/>
-<vertex x="17.272" y="49.022"/>
-<vertex x="80.01" y="49.022"/>
-<vertex x="80.264" y="48.768"/>
-<vertex x="80.264" y="13.462"/>
-<vertex x="80.772" y="12.954"/>
-<vertex x="96.012" y="10.16"/>
-<vertex x="96.012" y="-0.254"/>
-<vertex x="0" y="-0.254"/>
-</polygon>
 </signal>
 <signal name="VBB" class="1">
@@
 <wire x1="23.876" y1="62.992" x2="12.954" y2="62.992" width="1.27" layer="1"/>
 <wire x1="12.954" y1="62.992" x2="11.43" y2="65.532" width="1.27" layer="1"/>
-<wire x1="23.876" y1="62.672" x2="20.754" y2="59.55" width="0.4064" layer="1"/>
-<wire x1="20.754" y1="59.55" x2="16.15" y2="59.55" width="0.4064" layer="1"/>
+<wire x1="23.876" y1="62.672" x2="20.754" y2="59.55" width="0.6096" layer="1"/>
+<wire x1="20.754" y1="59.55" x2="16.15" y2="59.55" width="0.6096" layer="1"/>
 <wire x1="16.15" y1="59.55" x2="16.126" y2="59.526" width="0.4064" layer="1"/>
-<wire x1="16.126" y1="59.526" x2="16.126" y2="55.372" width="0.4064" layer="1"/>
+<wire x1="16.126" y1="59.526" x2="16.126" y2="55.372" width="0.6096" layer="1"/>
 <wire x1="23.876" y1="62.992" x2="24.992" y2="62.992" width="0.254" layer="1"/>
 <wire x1="24.992" y1="62.992" x2="25.7" y2="63.7" width="0.254" layer="1"/>
@@
 <wire x1="23.876" y1="58.166" x2="23.876" y2="60.772" width="1.27" layer="1"/>
 <wire x1="23.876" y1="60.772" x2="23.898" y2="60.75" width="0.4064" layer="1"/>
-<wire x1="23.898" y1="60.75" x2="26.7" y2="60.75" width="0.4064" layer="1"/>
-<wire x1="26.7" y1="60.75" x2="26.7" y2="64.4" width="0.4064" layer="1"/>
-<wire x1="26.7" y1="64.4" x2="26.45" y2="64.65" width="0.4064" layer="1"/>
-<wire x1="26.45" y1="64.65" x2="18.1" y2="64.65" width="0.4064" layer="1"/>
-<wire x1="18.1" y1="64.65" x2="17.218" y2="65.532" width="0.4064" layer="1"/>
+<wire x1="23.898" y1="60.75" x2="26.7" y2="60.75" width="0.6096" layer="1"/>
+<wire x1="26.7" y1="60.75" x2="26.7" y2="64.4" width="0.6096" layer="1"/>
+<wire x1="26.7" y1="64.4" x2="26.45" y2="64.65" width="0.6096" layer="1"/>
+<wire x1="26.45" y1="64.65" x2="18.1" y2="64.65" width="0.6096" layer="1"/>
+<wire x1="18.1" y1="64.65" x2="17.218" y2="65.532" width="0.6096" layer="1"/>
 <wire x1="17.218" y1="65.532" x2="16.256" y2="65.532" width="0.4064" layer="1"/>
 </signal>
@@
 </signal>
 </signals>
-<errors>
-</errors>
 </board>
 </drawing>

Commit message: minor fix, added teardrops
Routing:
- net GND: track 193.6 -> 275.2 mm
- net VDD: track 157.1 -> 218.8 mm
- net N$9: track 44.7 -> 88.7 mm
- net GH2B: track 49.8 -> 91.9 mm
- net GL2B: track 35.4 -> 69.8 mm
- net S2B: track 114.3 -> 146.3 mm
- net S1A: track 116.2 -> 145.4 mm
- net SENSE1: track 92.9 -> 121.8 mm
- net S1B: track 114.3 -> 142.9 mm
- net GL1A: track 31.9 -> 58.0 mm
- net ENABLE: track 60.7 -> 83.1 mm
- net N$13: track 40.3 -> 61.9 mm
- net N$12: track 19.4 -> 41.0 mm
- net N$14: track 24.3 -> 45.5 mm
- net REF: track 87.2 -> 107.2 mm
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Other:
- board text added: "OSHW"
- board text added: "v0.6.2"
- board text removed: "oshw.it"
- board text removed: "v0.6.1"

Commit message: REF fix
Connections:
- net REF: now also C5.1
- net VDD: no longer C5.1
Routing:
- net GND: track 275.2 -> 410.1 mm
- net REF: track 107.2 -> 137.0 mm, vias 2 -> 4
- net VDD: track 218.8 -> 239.2 mm
- net PFD2: track 37.9 -> 53.8 mm
- net MS2: track 52.8 -> 67.3 mm
- net GH2B: track 91.9 -> 106.1 mm
- net GL2B: track 69.8 -> 83.7 mm
- net PFD1: track 42.0 -> 55.8 mm
- net SENSE1: track 121.8 -> 135.0 mm
- net MS1: track 52.8 -> 65.8 mm
- net S1A: track 145.4 -> 156.4 mm
- net N$9: track 88.7 -> 99.7 mm
- net S2B: track 146.3 -> 156.3 mm
- net N$2: track 58.4 -> 67.9 mm
- net GL1B: track 49.9 -> 58.2 mm
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
Commit message: updated Creg footprint and value
Parts:
- C4: value 100u -> 1u; device rcl:153CLV-0605 -> rcl:153CLV-0405
Routing:
- net VBB: track 187.8 -> 203.1 mm, vias 2 -> 6
- net S1A: track 156.4 -> 169.0 mm
- net S2A: track 113.8 -> 126.1 mm
- net N$1: track 58.9 -> 51.1 mm
- net S2B: track 156.3 -> 162.0 mm, vias 4 -> 5
- net S1B: track 149.4 -> 153.1 mm, vias 4 -> 5
- net GND: track 410.1 -> 410.7 mm
- net RESET: track 78.7 -> 79.3 mm
